File: pcbs/encoder-optical-aedr8600/encoder-optical-aedr8600.kicad_sch (KiCad schematic)
At the start: 10 parts, among them J101 BM05B-GHS, U101 AEDR-8600-100

Commit message: Finish encoder-optical-aedr8600 PCB layout
Parts:
- C101: footprint Capacitor_SMD:C_0603_1608Metric -> Capacitor_SMD:C_0402_1005Metric
- R101: footprint Resistor_SMD:R_0603_1608Metric -> Resistor_SMD:R_0402_1005Metric
Changed lines of the file:
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@@
     (property "Reference" "R101" (id 0) (at 123.19 81.28 90))
     (property "Value" "180" (id 1) (at 123.19 83.82 90))
-    (property "Footprint" "Resistor_SMD:R_0603_1608Metric" (id 2) (at 123.19 89.408 90)
+    (property "Footprint" "Resistor_SMD:R_0402_1005Metric" (id 2) (at 123.19 89.408 90)
       (effects (font (size 1.27 1.27)) hide)
     )
@@
       (effects (font (size 1.27 1.27)) (justify left))
     )
-    (property "Footprint" "Capacitor_SMD:C_0603_1608Metric" (id 2) (at 157.1752 66.04 0)
+    (property "Footprint" "Capacitor_SMD:C_0402_1005Metric" (id 2) (at 157.1752 66.04 0)
       (effects (font (size 1.27 1.27)) hide)
     )
@@
     )
     (path "/c6c672db-068e-4740-ab56-9c092c78c067"
-      (reference "C101") (unit 1) (value "1u") (footprint "Capacitor_SMD:C_0603_1608Metric")
+      (reference "C101") (unit 1) (value "1u") (footprint "Capacitor_SMD:C_0402_1005Metric")
     )
     (path "/45c6ecd8-a666-483e-b413-617f0b8cd1b4"
@@
     )
     (path "/c25c6840-7de0-4db3-8816-c02818b30f6d"
-      (reference "R101") (unit 1) (value "180") (footprint "Resistor_SMD:R_0603_1608Metric")
+      (reference "R101") (unit 1) (value "180") (footprint "Resistor_SMD:R_0402_1005Metric")
     )
     (path "/e3edd19c-0408-44a8-a760-08b1389d72ad"
