File: pcbs/encoder-wheel-1/encoder-wheel-1.kicad_pcb (KiCad board)
At the start: 2 copper layers, 62 x 62 mm, 1 part

Commit message: Encoder wheel für Filmbelichtung angepasst und exportiert
Parts:
- added N101: Housing, encoder-wheel:code_wheel, F.Cu at (248.0, 48.0)
- added N101: Housing, encoder-wheel:code_wheel, F.Cu at (248.0, 129.0)
- added N101: Housing, encoder-wheel:code_wheel, F.Cu at (177.0, 48.0)
- added N101: Housing, encoder-wheel:code_wheel, F.Cu at (47.5, 129.0)
- added N101: Housing, encoder-wheel:code_wheel, F.Cu at (112.0, 129.0)
- added N101: Housing, encoder-wheel:code_wheel, F.Cu at (112.0, 48.0)
- added N101: Housing, encoder-wheel:code_wheel, F.Cu at (177.0, 129.0)
- moved N101 73.9 mm to (47.5, 48.0)
Other:
- board size 62 x 62 mm -> 262.5 x 143 mm
